Commit message: Update husky.urdf

File: Vehicles/husky/husky.urdf (robot description, URDF)
Before this commit: robot husky_robot, 11 links, 10 joints
Links:
- link base_link: geometry collision box size=1.0074 0.5709 0.2675; visual mesh filename=https://raw.githubusercontent.com/VallesMarinerisExplorer/E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
- link front_bumper_link: geometry visual mesh filename=https://raw.githubusercontent.com/VallesMarinerisExplorer/E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
- link front_left_wheel_link: geometry collision cylinder length=0.1143 radius=0.17775; visual mesh filename=https://raw.githubusercontent.com/VallesMarinerisExplorer/E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
- link front_right_wheel_link: geometry collision cylinder length=0.1143 radius=0.17775; visual mesh filename=https://raw.githubusercontent.com/VallesMarinerisExplorer/E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
- link rear_bumper_link: geometry visual mesh filename=https://raw.githubusercontent.com/VallesMarinerisExplorer/E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
- link rear_left_wheel_link: geometry collision cylinder length=0.1143 radius=0.17775; visual mesh filename=https://raw.githubusercontent.com/VallesMarinerisExplorer/E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
- link rear_right_wheel_link: geometry collision cylinder length=0.1143 radius=0.17775; visual mesh filename=https://raw.githubusercontent.com/VallesMarinerisExplorer/E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
- link top_plate_link: geometry visual mesh filename=https://raw.githubusercontent.com/VallesMarinerisExplorer/E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
- link user_rail_link: geometry visual mesh filename=https://raw.githubusercontent.com/VallesMarinerisExplorer/E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

Commit message: Update husky.urdf

File: Vehicles/husky/husky.urdf (robot description, URDF)
Before this commit: robot husky_robot, 11 links, 10 joints
Links:
- link base_link: geometry collision box size=1.0074 0.5709 0.2675; visual mesh filename=./meshes/base_link.stl
- link front_bumper_link: geometry visual mesh filename=./meshes/bumper.stl
- link front_left_wheel_link: geometry collision cylinder length=0.1143 radius=0.17775; visual mesh filename=./meshes/wheel.stl
- link front_right_wheel_link: geometry collision cylinder length=0.1143 radius=0.17775; visual mesh filename=./meshes/wheel.stl
- link rear_bumper_link: geometry visual mesh filename=./meshes/bumper.stl
- link rear_left_wheel_link: geometry collision cylinder length=0.1143 radius=0.17775; visual mesh filename=./meshes/wheel.stl
- link rear_right_wheel_link: geometry collision cylinder length=0.1143 radius=0.17775; visual mesh filename=./meshes/wheel.stl
- link top_plate_link: geometry visual mesh filename=./meshes/top_plate.stl
- link user_rail_link: geometry visual mesh filename=./meshes/user_rail.stl
